Commit message: ! adapted initial joint position to measured values

File: robots/reactor_description.URDF (robot description, URDF)
Before this commit: robot reactor_description, 7 links, 6 joints
Joints:
- joint elbow_pitch: limit lower=-3.141593 upper=0 effort=3.0 velocity=6.178465545 -> lower=-1.5708 upper=1.5708 effort=3.0 velocity=6.178465545; origin xyz=-0.1445 0 0.0385 rpy=0 0 0 -> xyz=-0.1445 0 0.0385 rpy=0 -1.48353 0
- joint shoulder_pitch: limit lower=0 upper=3.141593 effort=3.0 velocity=6.178465545 -> lower=-1.71042 upper=1.43117 effort=3.0 velocity=6.178465545; origin xyz=0 0 0.0265 rpy=0 0 0 -> xyz=0 0 0.0265 rpy=0 1.71042 0
- joint shoulder_yaw: limit lower=-3.141593 upper=3.141593 effort=1.5 velocity=6.178465545 -> lower=-2.61799 upper=2.61799 effort=1.5 velocity=6.178465545
- joint wrist_pitch: limit lower=-1.57079632679 upper=1.57079632679 effort=1.5 velocity=6.178465545 -> lower=-2.61799 upper=2.61799 effort=1.5 velocity=6.178465545
- joint wrist_roll: limit lower=-3.141593 upper=3.141593 effort=1.5 velocity=6.178465545 -> lower=-2.61799 upper=2.61799 effort=1.5 velocity=6.178465545

Commit message: ! removed CRs from lineendings

File: robots/reactor_description.URDF (robot description, URDF)
Before this commit: robot reactor_description, 7 links, 6 joints
Joints:
- joint elbow_pitch: origin xyz=-0.1445 0 0.0385 rpy=0 -1.48353 0 -> xyz=-0.1445 0 0.0385 rpy=0 -1.44862 0
- joint shoulder_pitch: origin xyz=0 0 0.0265 rpy=0 1.71042 0 -> xyz=0 0 0.0265 rpy=0 1.74533 0
