Commit message: ! added virtual dummy base link without inertia

File: robots/phantomx_reactor.urdf (robot description, URDF)
Before this commit: robot phantomx_reactor, 7 links, 6 joints
Links:
- added link virtual_base
Joints:
- added joint virtual_base_joint: type fixed, parent virtual_base, child base_link, origin xyz=0 0 0 rpy=0 0 0

Commit message: ! renamed base links (virtual and first non-virtual)

File: robots/phantomx_reactor.urdf (robot description, URDF)
Before this commit: robot phantomx_reactor, 8 links, 7 joints
Links:
- removed link virtual_base
- added link mounting_link, mass 0.33742; collision mesh filename=package://reactor_description/meshes/base_link_hull.STL; visual mesh filename=package://reactor_description/meshes/base_link.STL
- link base_link: mass 0.33742 -> None; geometry 
Joints:
- removed joint virtual_base_joint
- added joint base_joint: type fixed, parent base_link, child mounting_link, origin xyz=0 0 0 rpy=0 0 0
- joint shoulder_yaw: parent base_link -> mounting_link
